File: MixBoost.kicad_pcb (KiCad board)
At the start: 2 copper layers, 55 x 97 mm, 65 parts, among them J1 JACK_TRS_6PINS, J2 JACK_TRS_6PINS, J3 JACK_TRS_6PINS, P1 CONN_01X03, P2 CONN_01X03, P3 CONN_01X02, Q1 Q_NMOS_SGD, Q2 Q_NMOS_SGD, SW1 Switch_SPDT_x2, SW2 LAT/MOM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

Commit message: bump version to 0.96
Parts:
- removed R12: 100k, Resistors_SMD:R_0805_HandSoldering
Other:
- board text added: "mix/boost v0.96 by @mesotokyo http://meso .tokyo/"
- board text removed: "mix/boost v0.95 by @mesotokyo http://meso .tokyo/"
Changed lines of the file:
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@@
 (kicad_pcb (version 4) (host pcbnew 4.0.1-stable)
   (general
-    (links 145)
+    (links 143)
     (no_connects 0)
-    (area 97.711667 91.361666 156.325001 190.735)
+    (area 99.949999 92.949999 155.050001 190.050001)
     (thickness 1.6)
     (drawings 9)
     (tracks 791)
     (zones 0)
-    (modules 65)
+    (modules 64)
     (nets 55)
   )
   (page A4)
   (layers
-    (0 F.Cu signal hide)
-    (31 B.Cu signal hide)
+    (0 F.Cu signal)
+    (31 B.Cu signal)
     (32 B.Adhes user)
     (33 F.Adhes user)
@@
   )
   (setup
-    (last_trace_width 1)
+    (last_trace_width 0.25)
     (user_trace_width 1)
     (trace_clearance 0.25)
@@
   )
   (module Resistors_SMD:R_0805_HandSoldering (layer F.Cu)
-    (at 116.84 187.96 180)
-    (descr "Resistor SMD 0805, hand soldering")
-    (tags "resistor 0805")
-    (attr smd)
-    (fp_text reference R12 (at -1.66 1.46 180) (layer F.SilkS)
-      (effects (font (size 1 1) (thickness 0.15)))
-    )
-    (fp_text value 100k (at 0 1.75 180) (layer F.Fab)
-      (effects (font (size 1 1) (thickness 0.15)))
-    )
-    (fp_text user %R (at 0 0 180) (layer F.Fab)
-      (effects (font (size 0.5 0.5) (thickness 0.075)))
-    )
-    (fp_line (start -1 0.62) (end -1 -0.62) (layer F.Fab) (width 0.1))
-    (fp_line (start 1 0.62) (end -1 0.62) (layer F.Fab) (width 0.1))
-    (fp_line (start 1 -0.62) (end 1 0.62) (layer F.Fab) (width 0.1))
-    (fp_line (start -1 -0.62) (end 1 -0.62) (layer F.Fab) (width 0.1))
-    (fp_line (start 0.6 0.88) (end -0.6 0.88) (layer F.SilkS) (width 0.12))
-    (fp_line (start -0.6 -0.88) (end 0.6 -0.88) (layer F.SilkS) (width 0.12))
-    (fp_line (start -2.35 -0.9) (end 2.35 -0.9) (layer F.CrtYd) (width 0.05))
-    (fp_line (start -2.35 -0.9) (end -2.35 0.9) (layer F.CrtYd) (width 0.05))
-    (fp_line (start 2.35 0.9) (end 2.35 -0.9) (layer F.CrtYd) (width 0.05))
-    (fp_line (start 2.35 0.9) (end -2.35 0.9) (layer F.CrtYd) (width 0.05))
-    (pad 1 smd rect (at -1.35 0 180) (size 1.5 1.3) (layers F.Cu F.Paste F.Mask)
-      (net 13 "Net-(C17-Pad1)"))
-    (pad 2 smd rect (at 1.35 0 180) (size 1.5 1.3) (layers F.Cu F.Paste F.Mask)
-      (net 1 GND))
-    (model ${KISYS3DMOD}/Resistors_SMD.3dshapes/R_0805.wrl
-      (at (xyz 0 0 0))
-      (scale (xyz 1 1 1))
-      (rotate (xyz 0 0 0))
-    )
-  )
-  (module Resistors_SMD:R_0805_HandSoldering (layer F.Cu)
     (at 121.92 139.7 90)
     (descr "Resistor SMD 0805, hand soldering")
@@
     )
   )
-  (gr_text "mix/boost v0.95\nby @mesotokyo\nhttp://meso\n       .tokyo/" (at 134 97) (layer F.SilkS)
+  (gr_text "mix/boost v0.96\nby @mesotokyo\nhttp://meso\n       .tokyo/" (at 134 97) (layer F.SilkS)
     (effects (font (size 1 1) (thickness 0.2)) (justify left))
   )
