File: MixBoost.sch (KiCad schematic (older format))
At the start: 65 parts, among them J1 JACK_TRS_6PINS, J2 JACK_TRS_6PINS, J3 JACK_TRS_6PINS, P1 CONN_01X03, P2 CONN_01X03, P3 CONN_01X02, Q1 Q_NMOS_SGD, Q2 Q_NMOS_SGD, SW1 Switch_SPDT_x2, SW2 LAT/MOM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

Commit message: bump version to 0.96
Parts:
- removed R12: 100M, Resistors_SMD:R_0805_HandSoldering, symbol R
Changed lines of the file:
@@
-	1    0    0    -1
-$EndComp
-$Comp
-L R R12
-U 1 1 5984A602
-P 3250 3750
-F 0 "R12" V 3330 3750 50  0000 C CNN
-F 1 "100M" V 3250 3750 50  0000 C CNN
-F 2 "Resistors_SMD:R_0805_HandSoldering" V 3180 3750 50  0001 C CNN
-F 3 "" H 3250 3750 50  0000 C CNN
-	1    3250 3750
-	1    0    0    -1
-$EndComp
-$Comp
-L GND #PWR036
-U 1 1 5984A608
-P 3250 3900
-F 0 "#PWR036" H 3250 3650 50  0001 C CNN
-F 1 "GND" H 3250 3750 50  0000 C CNN
-F 2 "" H 3250 3900 50  0000 C CNN
-F 3 "" H 3250 3900 50  0000 C CNN
-	1    3250 3900
 	1    0    0    -1
 $EndComp
